File: cv_sequencer.kicad_pcb (KiCad board)
At the start: 4 copper layers, 111.3 x 22.4 mm, 106 parts, among them J1 :MIDI_IO, J10 PJ398SM, J11 PJ398SM, J12 PJ398SM, J13 PJ398SM, J2 SWD, J3 3086_Connector_Eurorack_Power, J4 3096_USBC_RA_SMD, J5 CV_OFFSET, J6 PJ398SM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

Commit message: Started re-route of PCB
Parts:
- removed J2: SWD, Shulltronics_Connectors:4005_SWD_Header
- added R39: 4008_Resistor_SMD_10k_0.125W_1%, Shulltronics_Generics:RES-0402, B.Cu at (137.6, 77.9)
- added TP1: GND, Shulltronics_Generics:TestPoint_Pad_D2.0mm, F.Cu at (160.2, 91.3)
- added U12: 4048_W25Q16JVSSIQ, Shulltronics_Integrated_Circuits:4048_16Mb_Flash_SOIC8, B.Cu at (140.1, 72.4)
- J10, J11, J12, J13, J6, J7, J8, J9: value PJ398SM -> 3085_MiniJack_Thonk_Vert
- U1: value 3097_TFT+SD_1.14in -> 3097_TFT_Display_SPI
- moved TP15 24.9 mm to (155.4, 90.9)
- moved TP16 24.0 mm to (151.3, 91.3)
- moved TP18 23.5 mm to (147.7, 91.6)
- moved J1 17.5 mm to (134.6, 55.9)
- moved U9 17.5 mm to (132.7, 59.4)
- moved R33 16.1 mm to (132.0, 62.5)
- moved R31 15.8 mm to (134.2, 62.4)
- moved R32 11.9 mm to (136.7, 62.4)
- moved R13 2.34 mm to (139.9, 77.9)
- moved C7 0.79 mm to (144.4, 76.5)
- moved C9 0.79 mm to (144.4, 77.6)
Connections:
- net Net-(R5-Pad1) renamed /QSPI_CS
- J4 pad B6: unconnected-(J4-PadB6) -> /USB_D+
- J4 pad B7: unconnected-(J4-PadB7) -> /USB_D-
- U2 pad 51: unconnected-(U2-Pad51) -> /QSPI_DATA3
- U2 pad 52: unconnected-(U2-Pad52) -> /QSPI_SCK
- U2 pad 53: unconnected-(U2-Pad53) -> /QSPI_DATA0
- U2 pad 54: unconnected-(U2-Pad54) -> /QSPI_DATA2
- U2 pad 55: unconnected-(U2-Pad55) -> /QSPI_DATA1
Routing:
- net /~{RESET}: track 74.4 -> 21.6 mm, vias 6 -> 5
- net /SWCLK: track 47.5 -> 0.94 mm, vias 2 -> 1
- net /SWDIO: track 46.0 -> 0.97 mm, vias 2 -> 1
- net /QSPI_CS: track 5.34 -> 21.9 mm
- net /QSPI_DATA2: track 0.00 -> 15.6 mm, vias 0 -> 2
- net /QSPI_DATA1: track 0.00 -> 14.8 mm
- net GND: track 28.7 -> 14.4 mm, vias 45 -> 42
- net /QSPI_DATA0: track 0.00 -> 11.7 mm, vias 0 -> 2
- net /QSPI_SCK: track 0.00 -> 10.9 mm, vias 0 -> 2
- net /LCD/SD_SDI: track 10.6 -> 0.00 mm
- net /UART_TX: track 10.5 -> 0.00 mm, vias 1 -> 0
- net /QSPI_DATA3: track 0.00 -> 9.97 mm, vias 0 -> 2
- net /UART_RX: track 9.51 -> 0.00 mm, vias 3 -> 0
- net /MIDI_SNK: track 9.30 -> 0.00 mm
- net /MIDI_OUT_SRC: track 8.72 -> 0.00 mm
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