File: cv_sequencer.kicad_sch (KiCad schematic)
At the start: 65 parts, among them J1 :MIDI_IO, J3 3086_Connector_Eurorack_Power, J4 3096_USBC_RA_SMD, SW1 RST, SW2 BOOT, U1 3097_TFT_Display_SPI, U10 PWR, U11 STAT, U2 4002_RP2040, U3 4032_Adjustable_Reg_200mA_SOT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

Commit message: Started re-route of PCB
Parts:
- gave numbers to parts that had none: 3
Connections:
- net VREG_1V2: now also C10.1, U2.50 (DVDD)
Changed lines of the file:
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@@
   (symbol (lib_id "Shulltronics_Passives:4008_Resistor_SMD_10k_0.125W_1%") (at 219.075 148.59 180) (unit 1)
     (in_bom yes) (on_board yes)
-    (property "Reference" "R?" (id 0) (at 216.535 148.59 90))
+    (property "Reference" "R39" (id 0) (at 216.535 148.59 90))
     (property "Value" "4008_Resistor_SMD_10k_0.125W_1%" (id 1) (at 213.995 154.94 90)
       (effects (font (size 1.27 1.27)) hide)
@@
   (symbol (lib_id "Shulltronics_ICs:4048_W25Q16JVSSIQ") (at 234.315 155.575 0) (unit 1)
     (in_bom yes) (on_board yes) (fields_autoplaced)
-    (property "Reference" "U?" (id 0) (at 236.3344 142.875 0)
+    (property "Reference" "U12" (id 0) (at 236.3344 142.875 0)
       (effects (font (size 1.27 1.27)) (justify left))
     )
@@
   (symbol (lib_id "Shulltronics_Sch_Symbols:GND") (at 234.315 165.735 0) (unit 1)
     (in_bom yes) (on_board yes)
-    (property "Reference" "#PWR?" (id 0) (at 234.315 172.085 0)
+    (property "Reference" "#PWR018" (id 0) (at 234.315 172.085 0)
       (effects (font (size 1.27 1.27)) hide)
     )
@@
   (symbol (lib_id "Shulltronics_Sch_Symbols:GND") (at 256.54 128.27 0) (unit 1)
     (in_bom yes) (on_board yes)
-    (property "Reference" "#PWR?" (id 0) (at 256.54 134.62 0)
+    (property "Reference" "#PWR031" (id 0) (at 256.54 134.62 0)
       (effects (font (size 1.27 1.27)) hide)
     )
@@
   (symbol (lib_id "Shulltronics_Sch_Symbols:VCC") (at 226.695 141.605 0) (unit 1)
     (in_bom yes) (on_board yes)
-    (property "Reference" "#PWR?" (id 0) (at 226.695 145.415 0)
+    (property "Reference" "#PWR017" (id 0) (at 226.695 145.415 0)
       (effects (font (size 1.27 1.27)) hide)
     )
@@
   (symbol (lib_id "Shulltronics_Sch_Symbols:TestPoint") (at 256.54 123.825 0) (unit 1)
     (in_bom yes) (on_board yes)
-    (property "Reference" "TP?" (id 0) (at 254.635 118.745 0)
+    (property "Reference" "TP1" (id 0) (at 254.635 118.745 0)
       (effects (font (size 1.27 1.27)) (justify left))
     )
@@
       (reference "#PWR016") (unit 1) (value "VSS") (footprint "")
     )
+    (path "/806390d5-8ed5-4b15-adcf-2e55d1a71f02"
+      (reference "#PWR017") (unit 1) (value "VCC") (footprint "")
+    )
+    (path "/4c18a907-ca0b-424b-85d0-506d67f17680"
+      (reference "#PWR018") (unit 1) (value "GND") (footprint "")
+    )
     (path "/ec75dbf9-36d4-4f80-84ea-bbeb4dadb453"
       (reference "#PWR019") (unit 1) (value "GND") (footprint "")
@@
       (reference "#PWR030") (unit 1) (value "VSS") (footprint "")
     )
+    (path "/5d898b00-d266-428d-a9b7-5eb01cdd924a"
+      (reference "#PWR031") (unit 1) (value "GND") (footprint "")
+    )
     (path "/a872c1aa-fae8-439b-8bc3-65de42b40b5b"
       (reference "#PWR0101") (unit 1) (value "GND") (footprint "")
@@
       (reference "#PWR0104") (unit 1) (value "VCC") (footprint "")
     )
-    (path "/4c18a907-ca0b-424b-85d0-506d67f17680"
-      (reference "#PWR?") (unit 1) (value "GND") (footprint "")
-    )
-    (path "/5d898b00-d266-428d-a9b7-5eb01cdd924a"
-      (reference "#PWR?") (unit 1) (value "GND") (footprint "")
-    )
-    (path "/806390d5-8ed5-4b15-adcf-2e55d1a71f02"
-      (reference "#PWR?") (unit 1) (value "VCC") (footprint "")
-    )
     (path "/eab8e027-9858-4087-bd40-ed8526d1e0e5"
       (reference "C1") (unit 1) (value "3089_Capacitor_100n_16V_0402") (footprint "Shulltronics_Generics:C_0402_HandSolder")
@@
     )
     (path "/26f99b10-df7a-42a7-aeda-632dd655d959"
-      (reference "R?") (unit 1) (value "4008_Resistor_SMD_10k_0.125W_1%") (footprint "Shulltronics_Generics:RES-0402")
+      (reference "R39") (unit 1) (value "4008_Resistor_SMD_10k_0.125W_1%") (footprint "Shulltronics_Generics:RES-0402")
     )
     (path "/fe47c086-eaa2-4714-b0d2-6fe34ddeaafa"
@@
       (reference "SW2") (unit 1) (value "BOOT") (footprint "Shulltronics_ElectroMechanical:4012_PushButton_NO_SMD")
     )
+    (path "/96d38b60-f73e-4b2a-977a-3fd1097da2eb"
+      (reference "TP1") (unit 1) (value "GND") (footprint "Shulltronics_Generics:TestPoint_Pad_D2.0mm")
+    )
     (path "/f37d5281-d51b-448e-b4fa-666b2af6d522"
       (reference "TP9") (unit 1) (value "3V1") (footprint "Shulltronics_Generics:TestPoint_Pad_D2.0mm")
@@
       (reference "TP28") (unit 1) (value "TRIG0") (footprint "Shulltronics_Generics:TestPoint_Pad_D2.0mm")
     )
-    (path "/96d38b60-f73e-4b2a-977a-3fd1097da2eb"
-      (reference "TP?") (unit 1) (value "GND") (footprint "Shulltronics_Generics:TestPoint_Pad_D2.0mm")
-    )
     (path "/74c75f18-4777-468f-90df-8c4e57ac4a0f"
       (reference "U1") (unit 1) (value "3097_TFT_Display_SPI") (footprint "Shulltronics-DevBoards:3097_TFT_Display_SPI")
@@
     )
     (path "/2bb5ccbe-f465-46c0-8890-a02e5cff0c30"
-      (reference "U?") (unit 1) (value "4048_W25Q16JVSSIQ") (footprint "Shulltronics_Integrated_Circuits:4048_16Mb_Flash_SOIC8")
+      (reference "U12") (unit 1) (value "4048_W25Q16JVSSIQ") (footprint "Shulltronics_Integrated_Circuits:4048_16Mb_Flash_SOIC8")
     )
     (path "/0ed7aa39-a4ef-4e9d-a8ce-bbafeb0d7fb6"
